Commit message: CAT

File: robocat.urdf (robot description, URDF)
Before this commit: robot robocat, 3 links, 2 joints
Links:
- added link backCylinder-leg; visual cylinder length=0.5 radius=0.1
- added link frontCylinder-leg; visual cylinder length=0.5 radius=0.1
- link backCylinder: mass None -> 5.0; geometry collision cylinder length=1.0 radius=0.2; visual cylinder length=1.0 radius=0.2
- link centerSphere: geometry visual sphere radius=0.1
- link frontCylinder: mass None -> 5.0
Joints:
- added joint backCylinder-leg-to-backCylinder: type fixed, parent backCylinder, child backCylinder-leg, origin xyz=0.0 -0.6 0.1
- added joint frontCylinder-leg-to-frontCylinder: type fixed, parent frontCylinder, child frontCylinder-leg, origin xyz=0.0 0.6 0.1
- joint back_to_center: axis 0 1 0 -> 0 0 1; limit lower=0.0 upper=1.507 effort=0.0 velocity=0.5 -> lower=-1.507 upper=1.507 effort=0.0 velocity=0.5
- joint front_to_center: limit lower=0.0 upper=1.507 effort=0.0 velocity=0.5 -> lower=-1.507 upper=1.507 effort=0.0 velocity=0.5
