Commit message: changes motors

File: cat.urdf (robot description, URDF)
Before this commit: robot physics, 2 links, 1 joints
Links:
- link back: geometry collision cylinder length=0.5 radius=0.1; visual cylinder length=1 radius=0.01
- link front: geometry collision cylinder length=0.5 radius=0.1; visual cylinder length=1 radius=0.01
